File: schematics&layouts/rc.brd (EAGLE design)
At the start: 99 x 51.7 mm, 17 parts, among them IC1 L293D, IC2 L293D, Q1 16MHz, U1 ATMEGA328P-PU

Commit message: updated eagle pcb schem
Parts:
- removed S1: SS12D07VG4, SS12D07VG4:SW_SS12D07VG4
- added SWITCH: (no value), pinhead:1X03
- turned MOTOR1 to 0 degrees
- renumbered 3.3V_VOLTAGE_REGU to 3.3V_REG, 5.5V_VOLTAGE_REGU to 5.5V_REG
Connections:
- removed net 3.3V: 3.3V_REG.3
- removed net CE: NRF.3
- removed net VCC: NRF.2
- new net +3.3V: 3.3V_REG.3, NRF.2, NRF.3
- net GND: now also SWITCH.3; no longer S1.2, S1.3
- net N$21: now also SWITCH.1; no longer S1.1
- net VCC_2: now also SWITCH.2
Routing:
- net +3.3V: track 0.00 -> 58.1 mm, vias 0 -> 1
- net GND: track 270.3 -> 221.7 mm, vias 1 -> 0
- net GND1: track 101.5 -> 77.4 mm
- net N$8: track 110.8 -> 88.2 mm, vias 1 -> 0
- net GND3: track 90.6 -> 80.0 mm
- net IRQ: track 31.8 -> 22.0 mm
- net N$11: track 40.8 -> 50.2 mm
- net N$21: track 86.8 -> 95.2 mm
- net N$19: track 24.5 -> 31.2 mm
- net N$10: track 92.8 -> 86.3 mm
- net 5V: track 134.7 -> 128.5 mm, vias 0 -> 1
- net N$3: track 110.7 -> 104.6 mm
- net N$17: track 26.0 -> 32.0 mm
- net SCK: track 17.8 -> 23.5 mm
- net N$20: track 24.4 -> 30.1 mm
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Other:
- board size 99 x 51.7 mm -> 96.5 x 51.7 mm
- board text added: "Vroom Vroom"
- board text added: "YO BOI GED"

Commit message: update schematic
Parts:
- added 3VL, 5VL, BOOTUP: (no value), led:LED5MM
- added J1: 10103594, Connector_USB:10103594
- added JP1: SPI+RESET, pinhead:1X04
- added R1: 50Ω, rcl:0204/7
- added R2, R3: 150Ω, rcl:0204/7
- added U$1: CH340C, CH340C:SOP16-1.27-10.0X5.0MM
- POWER: value (none) -> BLOCK; device pinhead:1X02 -> Connector:TERMBLK_254-2N
- turned POWER to 270 degrees
Connections:
- new net N$22: 5VL.K, R2.2
- new net N$23: 3VL.K, R1.2
- new net N$24: J1.2, U$1.6
- new net N$25: JP1.1, U1.1
- new net N$26: J1.3, U$1.5
- new net N$29: J1.1, U$1.4
- net +3.3V: now also 3VL.A
- net 5V: now also 5VL.A
- net GND: now also BOOTUP.K, J1.5, R1.1, R2.1, R3.1, R3.2, U$1.1; no longer SWITCH.3
- net MISO: now also JP1.3
- net MOSI: now also JP1.4
- net N$18: now also U$1.2
- net N$2: now also U$1.3
- net SCK: now also BOOTUP.A, JP1.2
Routing:
- net GND: track 221.7 -> 207.4 mm
- net N$21: track 95.2 -> 92.5 mm
- net VCC_2: track 127.2 -> 125.4 mm
Other:
- board text removed: "Vroom Vroom"
- board text removed: "YO BOI GED"

Commit message: updated schm
Parts:
- moved BOOTUP 87.0 mm to (78.7, 61.0)
- moved JP1 83.9 mm to (48.3, 59.7)
- moved R3 82.9 mm to (67.3, 57.1)
- moved 5VL 77.5 mm to (106.7, 19.1)
- moved U$1 61.7 mm to (52.1, 17.8), turned to 0 degrees
- moved R1 55.5 mm to (85.1, 14.0)
- moved J1 50.7 mm to (33.0, 24.1), turned to 270 degrees
- moved R2 46.0 mm to (73.7, 12.7)
- moved MOTOR3 12.7 mm to (120.7, 11.4)
- moved MOTOR4 8.89 mm to (120.7, 63.5)
- moved MOTOR1 6.48 mm to (34.3, 12.7)
- moved C2 5.08 mm to (64.8, 29.2)
- moved 3.3V_REG 4.58 mm to (88.9, 33.0)
- moved POWER 4.02 mm to (119.4, 22.9)
- moved C1 3.81 mm to (76.2, 29.2)
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Connections:
- net N$7: now also MOTOR1.2; no longer MOTOR1.1
- net N$8: now also MOTOR1.1; no longer MOTOR1.2
Routing:
- net GND: track 207.4 -> 324.7 mm, vias 0 -> 2
- net SCK: track 23.5 -> 78.8 mm, vias 0 -> 1
- net MOSI: track 15.2 -> 66.1 mm, vias 0 -> 1
- net N$18: track 13.4 -> 55.9 mm, vias 0 -> 1
- net MISO: track 27.5 -> 68.5 mm, vias 0 -> 1
- net N$26: track 0.00 -> 40.7 mm
- net 5V: track 128.5 -> 167.3 mm
- net N$29: track 0.00 -> 34.4 mm
- net N$22: track 0.00 -> 33.1 mm
- net N$25: track 0.00 -> 32.5 mm, vias 0 -> 1
- net N$8: track 88.2 -> 119.7 mm
- net +3.3V: track 58.1 -> 86.9 mm
- net N$24: track 0.00 -> 24.6 mm, vias 0 -> 2
- net N$7: track 102.1 -> 121.9 mm
- net N$2: track 21.2 -> 41.0 mm, vias 0 -> 1
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Other:
- board size 96.5 x 51.7 mm -> 97.8 x 60.6 mm

Commit message: Updated
Parts:
- removed 3.3V_REG: HT7333, HT7333:IC_HT7333
- removed RX_TX: (no value), pinhead:1X02
- removed SWITCH: (no value), pinhead:1X03
- added SWITCH-VCC: DS02E, Switch:DS-02
- added TX_RX: (no value), pinhead:1X02
- added U2: LM1117T-3.3, LM1117T-3.3:TO254P470X1016X2222-3P
- MOTOR1: value (none) -> AYE AM WALKIN' HERE
- MOTOR2: value (none) -> YO BOI GED
- moved R2 22.9 mm to (96.5, 14.0)
- moved JP1 11.4 mm to (58.4, 64.8)
- moved 3VL 8.98 mm to (85.1, 20.3)
- moved Q1 8.03 mm to (69.8, 14.0)
- moved U$1 7.73 mm to (50.8, 25.4)
- moved R3 6.84 mm to (73.7, 54.6)
- moved BOOTUP 5.68 mm to (73.7, 63.5)
- moved NRF 5.24 mm to (92.7, 55.9)
- moved R1 3.59 mm to (87.6, 11.4)
- moved J1 1.27 mm to (31.8, 24.1)
- moved 5VL 1.27 mm to (106.7, 20.3)
Connections:
- removed net GND4: IC1.12
- removed net N$18: RX_TX.2, U$1.2, U1.2
- removed net N$2: RX_TX.1, U$1.3, U1.3
- new net N$27: POWER.1, SWITCH-VCC.2
- new net N$28: SWITCH-VCC.4, U1.7
- new net N$31: J1.5, U$1.1
- new net N$32: IC1.15, U1.5
- new net N$33: IC1.7, U1.25
- new net N$34: IC2.7, U1.15
- new net N$35: IC2.2, U1.16
- new net RX: TX_RX.2, U$1.2, U1.2
- new net TX: TX_RX.1, U$1.3, U1.3
- net +3.3V: now also U2.2; no longer 3.3V_REG.3
- net 5V: now also SWITCH-VCC.1, U2.3; no longer 3.3V_REG.2, U1.7
- net GND: now also IC1.12, U2.1; no longer 3.3V_REG.1, IC1.5, J1.5, R3.1, R3.2, U$1.1
- net GND2: now also IC1.5
- net N$12: no longer IC2.2
- net N$14: no longer IC2.7
- net N$15: no longer IC1.7
- net N$16: no longer IC1.15
- net N$21: now also BOOTUP.A, R3.2; no longer POWER.1, SWITCH.1
- net SCK: now also R3.1; no longer BOOTUP.A
- net VCC_2: now also SWITCH-VCC.3; no longer SWITCH.2
Routing:
- net GND: track 324.7 -> 228.1 mm
- net GND2: track 0.00 -> 93.7 mm, vias 0 -> 1
- net N$21: track 98.3 -> 11.0 mm
- net N$28: track 0.00 -> 60.0 mm
- net N$18: track 55.9 -> 0.00 mm, vias 1 -> 0
- net +3.3V: track 86.9 -> 41.1 mm, vias 1 -> 0
- net N$27: track 0.00 -> 45.2 mm
- net N$32: track 0.00 -> 44.4 mm, vias 0 -> 1
- net N$2: track 41.0 -> 0.00 mm, vias 1 -> 0
- net N$7: track 121.9 -> 84.6 mm
- net SCK: track 78.8 -> 45.1 mm, vias 1 -> 0
- net RX: track 0.00 -> 33.1 mm
- net N$34: track 0.00 -> 30.0 mm
- net TX: track 0.00 -> 26.6 mm, vias 0 -> 1
- net N$33: track 0.00 -> 26.1 mm
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
Commit message: updated enviroment configuration for usbasp
Parts:
- removed BOOTUP: (no value), led:LED5MM
- removed JP1: SPI+RESET, pinhead:1X04
- removed R3: 150Ω, rcl:0204/7
- added 3VTP, 5VTP, GNDTP, VCC2TP: TPB1,27, testpad:B1,27
- added PROGRAM_ME: ICSP, pinhead:2X03
- MOTOR1: value AYE AM WALKIN' HERE -> B2B-XH-A; device pinhead:1X02 -> Connector:B2B-XH-A
- MOTOR2: value YO BOI GED -> B2B-XH-A; device pinhead:1X02 -> Connector:B2B-XH-A
- MOTOR3, MOTOR4: value (none) -> B2B-XH-A; device pinhead:1X02 -> Connector:B2B-XH-A
- moved MOTOR3 52.1 mm to (119.4, 63.5), turned to 0 degrees
- moved MOTOR4 49.5 mm to (119.4, 14.0)
- moved NRF 9.92 mm to (85.1, 62.2)
- moved POWER 3.81 mm to (119.4, 26.7)
- moved TX_RX 3.59 mm to (55.9, 35.6)
- moved MOTOR1 2.84 mm to (31.8, 14.0)
- moved I2C 1.80 mm to (45.7, 34.3)
- moved MOTOR2 1.27 mm to (31.8, 63.5)
Connections:
- removed net N$21: BOOTUP.A, R3.2
- removed net N$25: JP1.1, U1.1
- new net RESET: PROGRAM_ME.5, U1.1
- net +3.3V: now also 3VTP.TP
- net 5V: now also 5VTP.TP, PROGRAM_ME.2
- net GND: now also GNDTP.TP, PROGRAM_ME.6; no longer BOOTUP.K
- net MISO: now also PROGRAM_ME.1; no longer JP1.3
- net MOSI: now also PROGRAM_ME.4; no longer JP1.4
- net N$28: now also U$1.16
- net N$3: now also MOTOR3.1; no longer MOTOR4.1
- net N$4: now also MOTOR3.2; no longer MOTOR4.2
- net N$5: now also MOTOR4.1; no longer MOTOR3.1
- net N$6: now also MOTOR4.2; no longer MOTOR3.2
- net SCK: now also PROGRAM_ME.3; no longer JP1.2, R3.1
- net VCC_2: now also VCC2TP.TP
Routing:
- net 5V: track 155.9 -> 205.3 mm, vias 0 -> 1
- net N$28: track 60.0 -> 95.6 mm, vias 0 -> 2
- net RESET: track 0.00 -> 32.5 mm
- net +3.3V: track 41.1 -> 69.1 mm
- net N$25: track 24.6 -> 0.00 mm
- net GND: track 228.1 -> 243.7 mm, vias 2 -> 3
- net N$21: track 11.0 -> 0.00 mm
- net IRQ: track 17.5 -> 26.1 mm
- net MISO: track 45.1 -> 52.7 mm, vias 0 -> 1
- net VCC_2: track 135.5 -> 140.3 mm
- net MOSI: track 43.1 -> 47.9 mm, vias 0 -> 1
- net N$6: track 104.4 -> 108.7 mm
- net SCK: track 45.1 -> 49.1 mm
- net N$27: track 45.2 -> 42.8 mm
- net N$7: track 84.6 -> 86.5 mm
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
Commit message: updated schematic
Parts:
- removed 3VTP, 5VTP, GNDTP, VCC2TP: TPB1,27, testpad:B1,27
- removed PROGRAM_ME: ICSP, pinhead:2X03
- added ICSP: (no value), pinhead:2X05
- moved R2 6.84 mm to (102.9, 11.4)
- moved C2 6.84 mm to (71.1, 26.7)
- moved TX_RX 6.48 mm to (62.2, 34.3)
- moved Q1 6.35 mm to (74.9, 17.8)
- moved 3VL 6.35 mm to (91.4, 20.3)
- moved NRF 3.81 mm to (81.3, 62.2)
- moved C1 3.59 mm to (78.7, 26.7)
- moved R1 2.54 mm to (90.2, 11.4)
- moved 5VL 1.27 mm to (105.4, 20.3)
Connections:
- removed net N$29: J1.1, U$1.4
- new net N$2: J1.1, U$1.16
- net +3.3V: no longer 3VTP.TP
- net 5V: now also ICSP.6; no longer 5VTP.TP, PROGRAM_ME.2
- net GND: now also ICSP.10; no longer GNDTP.TP, PROGRAM_ME.6
- net MISO: now also ICSP.5; no longer PROGRAM_ME.1
- net MOSI: now also ICSP.8; no longer PROGRAM_ME.4
- net N$28: no longer U$1.16
- net RESET: now also ICSP.9; no longer PROGRAM_ME.5
- net SCK: now also ICSP.7; no longer PROGRAM_ME.3
- net VCC_2: no longer VCC2TP.TP
Routing:
- net GND: track 243.7 -> 0.00 mm, vias 3 -> 0
- net 5V: track 205.3 -> 0.00 mm, vias 1 -> 0
- net N$28: track 95.6 -> 53.1 mm, vias 2 -> 0
- net N$6: track 108.7 -> 140.5 mm
- net N$7: track 86.5 -> 111.9 mm
- net N$29: track 23.1 -> 0.00 mm
- net N$5: track 105.5 -> 125.9 mm
- net +3.3V: track 69.1 -> 50.6 mm
- net GND1: track 102.1 -> 83.8 mm
- net N$8: track 102.8 -> 119.0 mm
- net N$14: track 58.9 -> 74.6 mm, vias 1 -> 0
- net N$2: track 0.00 -> 14.1 mm
- net N$15: track 54.3 -> 68.1 mm
- net RESET: track 32.5 -> 20.3 mm
- net N$32: track 44.4 -> 54.9 mm, vias 1 -> 0
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- added copper zone on layer 15, net 5V
- added copper zone on layer 2, net GND
